File: powermod.kicad_sch (KiCad schematic)
At the start: 20 parts, among them J1 Conn_02x07_Odd_Even, J2 Conn_02x07_Odd_Even, U1 TPS54260DGQ

Commit message: feat: 1.4
Other:
- title: powermod-tps54260-1.2 -> powermod-tps54260-1.4
Changed lines of the file:
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@@
 	(paper "A4")
 	(title_block
-		(title "powermod-tps54260-1.2")
+		(title "powermod-tps54260-1.4")
 		(company "Lightside Instruments AS")
 	)
